File: PCB/esp32_only/pixo_esp.kicad_pcb (KiCad board)
At the start: 2 copper layers, 75 x 75 mm, 53 parts, among them J1 PIXO_CONN, P1 USB_OTG, P2 GPIO, SW2 GPIO0, SW3 RESET, U1 AP2112K-3.3V, U3 FT230XS, U4 ESP-32S

Commit message: added accelerometer, changed GPIO
Parts:
- added J2: ACC, Pin_Headers:Pin_Header_Straight_1x08, F.Cu at (106.5, 120.3)
- moved REF** 0.07 mm to (105.8, 125.2)
- moved REF** 0.07 mm to (123.6, 125.2)
- moved REF** 0.07 mm to (108.4, 125.2)
- moved REF** 0.07 mm to (103.3, 125.2)
- moved REF** 0.07 mm to (100.8, 125.2)
- moved REF** 0.07 mm to (121.1, 125.2)
- moved REF** 0.07 mm to (118.5, 125.2)
- moved REF** 0.07 mm to (116.0, 125.2)
- moved REF** 0.07 mm to (113.5, 125.2)
- moved REF** 0.07 mm to (110.9, 125.2)
Connections:
- net /GPIO14_A6 renamed INT
- net /SCL renamed SCL
- net /SDA renamed SDA
- P2 pad 10: /GPIO15_A8 -> /GPIO17
- P2 pad 9: /GPIO13_A12 -> /GPIO16
- U4 pad 27: Net-(U4-Pad27) -> /GPIO16
- U4 pad 28: Net-(U4-Pad28) -> /GPIO17
Routing:
- net /GPIO17: track 0.00 -> 38.2 mm, vias 0 -> 2
- net /GPIO16: track 0.00 -> 36.6 mm, vias 0 -> 2
- net SDA: track 56.4 -> 92.0 mm
- net INT: track 18.8 -> 52.1 mm
- net /GPIO15_A8: track 31.9 -> 0.00 mm
- net SCL: track 52.6 -> 83.5 mm
- net /GPIO13_A12: track 23.1 -> 0.00 mm
- net +3V3: track 132.6 -> 138.1 mm
Other:
- board text added: "AD0"
- board text added: "INT"
- board text added: "IO14/A6/ACC_INT"
- board text added: "IO16"
- board text added: "IO17"
- board text added: "PIXO_RGB V0.1a IDLE HANDS DEV."
- board text removed: "IO13/A12"
- board text removed: "IO14/A6"
- board text removed: "IO15/A8"
- board text removed: "PIXO_RGB V0.1p IDLE HANDS DEV."
