File: PCB/esp32_only/pixo_esp.kicad_pcb (KiCad board)
At the start: 2 copper layers, 75 x 75 mm, 54 parts, among them J1 PIXO_CONN, J2 ACC, P1 USB_OTG, P2 GPIO, SW2 GPIO0, SW3 RESET, U1 AP2112K-3.3V, U3 FT230XS, U4 ESP-32S

Commit message: changed led pad layout
Routing:
- net GND: track 49.1 -> 50.5 mm, vias 26 -> 27
Other:
- board text added: "/100"
- board text added: "BOOT"
- board text added: "PIXO Pixel Make/100 Project"
Changed lines of the file:
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@@
     (area 59.425 63.6 186.475001 188.195005)
     (thickness 1.6)
-    (drawings 39)
-    (tracks 392)
+    (drawings 42)
+    (tracks 395)
     (zones 0)
     (modules 54)
@@
     (visible_elements 7FFFEF7F)
     (pcbplotparams
-      (layerselection 0x010f4_80000001)
+      (layerselection 0x010f8_80000001)
       (usegerberextensions false)
       (excludeedgelayer true)
@@
       (effects (font (size 1.5 1.5) (thickness 0.15)))
     )
-    (fp_text value RESET (at -2 -3.75 270) (layer F.SilkS)
-      (effects (font (size 0.5 0.5) (thickness 0.125)))
+    (fp_text value RESET (at -6.03 -0.08 360) (layer F.SilkS)
+      (effects (font (size 1.5 1.5) (thickness 0.125)))
     )
     (fp_line (start -2.6 -3.2) (end 2.8 -3.2) (layer F.SilkS) (width 0.15))
@@
     )
   )
+  (gr_text /100 (at 136.76 164.75) (layer B.SilkS)
+    (effects (font (size 3 3) (thickness 0.5)) (justify mirror))
+  )
+  (gr_text "PIXO Pixel\nMake/100 Project" (at 150.08 154.31) (layer B.SilkS)
+    (effects (font (size 2 2) (thickness 0.3)) (justify mirror))
+  )
+  (gr_text BOOT (at 167.55 106.16) (layer F.SilkS)
+    (effects (font (size 1.5 1.5) (thickness 0.3)))
+  )
   (gr_text 3V3 (at 124.3 117.45 90) (layer F.SilkS)
     (effects (font (size 1 1) (thickness 0.25)))
@@
   (gr_circle (center 169.00058 169.000169) (end 170.60058 169.000169) (layer Edge.Cuts) (width 0.1))
   (gr_arc (start 125.5 157.6) (end 126 157.6) (angle -90.000003) (layer Edge.Cuts) (width 0.1))
+  (segment (start 121.5 107.98) (end 121.5 109.29) (width 0.2) (layer F.Cu) (net 1))
+  (segment (start 121.5 109.29) (end 121.46 109.33) (width 0.2) (layer F.Cu) (net 1))
+  (via (at 121.46 109.33) (size 0.6) (drill 0.4) (layers F.Cu B.Cu) (net 1))
   (segment (start 98.81 116.975) (end 98.81 112.96) (width 0.4) (layer F.Cu) (net 1))
   (segment (start 98.81 112.96) (end 98.75 112.9) (width 0.4) (layer F.Cu) (net 1))
