File: PCB/esp32_only/pixo_esp.sch (KiCad schematic (older format))
At the start: 35 parts, among them J1 PIXO_CONN, P1 USB_OTG, P2 GPIO, SW2 GPIO0, SW3 RESET, U1 AP2112K-3.3V, U3 FT230XS, U4 ESP-32S

Commit message: added accelerometer, changed GPIO
Parts:
- added J2: ACC, Pin_Headers:Pin_Header_Straight_1x08, symbol Conn_01x08
Connections:
- net labels added: AD0, GPIO16, GPIO17, INT, XCL, XDA
- wire segments 122 -> 135
Other:
- note added: "Acceleromter(MPU6050)"
- moved on the sheet: J1, P2
Changed lines of the file:
@@
 Wire Wire Line
 	7300 5200 7450 5200
-Text GLabel 2350 5750 0    39   Input ~ 0
+Text GLabel 1800 5600 0    39   Input ~ 0
 CKS
-Text GLabel 2350 5850 0    39   Input ~ 0
+Text GLabel 1800 5700 0    39   Input ~ 0
 SDS
 Wire Wire Line
-	2350 5650 2300 5650
+	1800 5500 1750 5500
 $Comp
 L GND #PWR021
 U 1 1 5A5EF462
-P 2300 6000
-F 0 "#PWR021" H 2300 5750 50  0001 C CNN
-F 1 "GND" H 2300 5850 50  0000 C CNN
-F 2 "" H 2300 6000 50  0000 C CNN
-F 3 "" H 2300 6000 50  0000 C CNN
-	1    2300 6000
-	1    0    0    -1
-$EndComp
-Wire Wire Line
-	2350 5950 2300 5950
-Wire Wire Line
-	2300 5950 2300 6000
+P 1750 5850
+F 0 "#PWR021" H 1750 5600 50  0001 C CNN
+F 1 "GND" H 1750 5700 50  0000 C CNN
+F 2 "" H 1750 5850 50  0000 C CNN
+F 3 "" H 1750 5850 50  0000 C CNN
+	1    1750 5850
+	1    0    0    -1
+$EndComp
+Wire Wire Line
+	1800 5800 1750 5800
+Wire Wire Line
+	1750 5800 1750 5850
 $Comp
 L Conn_01x04 J1
 U 1 1 5A5EF625
-P 2550 5850
-F 0 "J1" H 2550 6050 50  0000 C CNN
-F 1 "PIXO_CONN" H 2550 5550 50  0000 C CNN
-F 2 "Connectors_JST_PH:Connectors_JST_S4B-PH-SM4-TB" H 2550 5850 50  0001 C CNN
-F 3 "" H 2550 5850 50  0001 C CNN
-F 4 "455-1751-1-ND" H 2550 5850 60  0001 C CNN "Digikey Part No."
-	1    2550 5850
+P 2000 5700
+F 0 "J1" H 2000 5900 50  0000 C CNN
+F 1 "PIXO_CONN" H 2000 5400 50  0000 C CNN
+F 2 "Connectors_JST_PH:Connectors_JST_S4B-PH-SM4-TB" H 2000 5700 50  0001 C CNN
+F 3 "" H 2000 5700 50  0001 C CNN
+F 4 "455-1751-1-ND" H 2000 5700 60  0001 C CNN "Digikey Part No."
+	1    2000 5700
 	1    0    0    1
 $EndComp
-Text GLabel 2300 5650 0    59   Input ~ 0
+Text GLabel 1750 5500 0    59   Input ~ 0
 VSPLY
 Text Notes 3000 1050 0    157  ~ 0
@@
 Text Label 4650 4350 1    59   ~ 0
 GPIO15_A8
-Text Notes 3250 5350 0    98   ~ 0
+Text Notes 2700 5200 0    98   ~ 0
 GPIO32
 Wire Wire Line
-	3750 6250 3500 6250
-Wire Wire Line
-	3750 6350 3500 6350
-Wire Wire Line
-	3750 5950 3500 5950
-Wire Wire Line
-	3750 6050 3500 6050
-Wire Wire Line
-	3750 5750 3500 5750
-Wire Wire Line
-	3750 5850 3500 5850
-Text Label 3750 6650 0    59   ~ 0
+	3200 6100 2950 6100
+Wire Wire Line
+	3200 6200 2950 6200
+Wire Wire Line
+	3200 5800 2950 5800
+Wire Wire Line
+	3200 5900 2950 5900
+Wire Wire Line
+	3200 5600 2950 5600
+Wire Wire Line
+	3200 5700 2950 5700
+Text Label 3200 6500 0    59   ~ 0
 GPIO32_A7
-Text Label 3750 6550 0    59   ~ 0
+Text Label 3200 6400 0    59   ~ 0
 GPIO33_A9
-Text Label 3750 6450 0    59   ~ 0
+Text Label 3200 6300 0    59   ~ 0
 A1_DAC1
-Text Label 3750 6350 0    59   ~ 0
+Text Label 3200 6200 0    59   ~ 0
 A0_DAC2
-Text Label 3750 6250 0    59   ~ 0
+Text Label 3200 6100 0    59   ~ 0
 GPIO14_A6
-Text Label 3750 6150 0    59   ~ 0
+Text Label 3200 6000 0    59   ~ 0
 GPIO12_A11
 Wire Wire Line
-	3500 6450 3750 6450
-Wire Wire Line
-	3500 6150 3750 6150
-Text Label 3750 6050 0    59   ~ 0
-GPIO13_A12
-Wire Wire Line
-	3500 6550 3750 6550
-Wire Wire Line
-	3500 6650 3750 6650
-Text Label 3750 5950 0    59   ~ 0
-GPIO15_A8
-Text Label 3750 5850 0    59   ~ 0
+	2950 6300 3200 6300
+Wire Wire Line
+	2950 6000 3200 6000
+Text Label 3200 5900 0    59   ~ 0
+GPIO16
+Wire Wire Line
+	2950 6400 3200 6400
+Wire Wire Line
+	2950 6500 3200 6500
+Text Label 3200 5800 0    59   ~ 0
+GPIO17
+Text Label 3200 5700 0    59   ~ 0
 SCL
-Text Label 3750 5750 0    59   ~ 0
+Text Label 3200 5600 0    59   ~ 0
 SDA
 $Comp
 L CONN_01X12 P2
 U 1 1 5A5F5313
-P 3300 6300
-F 0 "P2" H 3300 6950 50  0000 C CNN
-F 1 "GPIO" V 3400 6300 50  0000 C CNN
-F 2 "Pin_Headers:Pin_Header_Straight_1x12" H 3300 6300 50  0001 C CNN
-F 3 "" H 3300 6300 50  0000 C CNN
-	1    3300 6300
+P 2750 6150
+F 0 "P2" H 2750 6800 50  0000 C CNN
+F 1 "GPIO" V 2850 6150 50  0000 C CNN
+F 2 "Pin_Headers:Pin_Header_Straight_1x12" H 2750 6150 50  0001 C CNN
+F 3 "" H 2750 6150 50  0000 C CNN
+	1    2750 6150
 	-1   0    0    1
 $EndComp
 Wire Wire Line
-	3500 6750 3750 6750
-Wire Wire Line
-	3500 6850 3750 6850
+	2950 6600 3200 6600
+Wire Wire Line
+	2950 6700 3200 6700
 $Comp
 L +3.3V #PWR029
 U 1 1 5A5F5DFB
-P 3750 6750
-F 0 "#PWR029" H 3750 6600 50  0001 C CNN
-F 1 "+3.3V" H 3750 6890 50  0000 C CNN
-F 2 "" H 3750 6750 60  0000 C CNN
-F 3 "" H 3750 6750 60  0000 C CNN
-	1    3750 6750
+P 3200 6600
+F 0 "#PWR029" H 3200 6450 50  0001 C CNN
+F 1 "+3.3V" H 3200 6740 50  0000 C CNN
+F 2 "" H 3200 6600 60  0000 C CNN
+F 3 "" H 3200 6600 60  0000 C CNN
+	1    3200 6600
 	0    1    1    0
 $EndComp
@@
 L GND #PWR030
 U 1 1 5A5F5E6F
-P 3750 6850
-F 0 "#PWR030" H 3750 6600 50  0001 C CNN
-F 1 "GND" H 3750 6700 50  0000 C CNN
-F 2 "" H 3750 6850 60  0000 C CNN
-F 3 "" H 3750 6850 60  0000 C CNN
-	1    3750 6850
+P 3200 6700
+F 0 "#PWR030" H 3200 6450 50  0001 C CNN
+F 1 "GND" H 3200 6550 50  0000 C CNN
+F 2 "" H 3200 6700 60  0000 C CNN
+F 3 "" H 3200 6700 60  0000 C CNN
+	1    3200 6700
 	0    -1   -1   0
 $EndComp
+$Comp
+L Conn_01x08 J2
+U 1 1 5A8DAF78
+P 4900 6000
+F 0 "J2" H 4900 6400 50  0000 C CNN
+F 1 "ACC" H 4900 5500 50  0000 C CNN
+F 2 "Pin_Headers:Pin_Header_Straight_1x08" H 4900 6000 50  0001 C CNN
+F 3 "" H 4900 6000 50  0001 C CNN
+	1    4900 6000
+	-1   0    0    1
+$EndComp
+Wire Wire Line
+	5100 6300 5150 6300
+Wire Wire Line
+	5100 6200 5150 6200
+Wire Wire Line
+	5100 6100 5150 6100
+Wire Wire Line
+	5100 6000 5150 6000
+Wire Wire Line
+	5100 5900 5150 5900
+Wire Wire Line
+	5100 5800 5150 5800
+Wire Wire Line
+	5100 5700 5450 5700
+Wire Wire Line
+	5100 5600 5300 5600
+Text GLabel 5150 6300 2    39   Input ~ 0
+INT
+Text GLabel 5150 6200 2    39   Input ~ 0
+AD0
+Text GLabel 5150 6100 2    39   Input ~ 0
+XCL
+Text GLabel 5150 6000 2    39   Input ~ 0
+XDA
+Text GLabel 5150 5900 2    39   Input ~ 0
+SDA
+Text GLabel 5150 5800 2    39   Input ~ 0
+SCL
+Text GLabel 5600 6800 2    39   Input ~ 0
+INT
+Text GLabel 5600 6700 2    39   Input ~ 0
+SDA
+Text GLabel 5600 6600 2    39   Input ~ 0
+SCL
+Wire Wire Line
+	5600 6600 5450 6600
+Wire Wire Line
+	5600 6700 5450 6700
+Wire Wire Line
+	5600 6800 5450 6800
+Text Label 5450 6800 2    59   ~ 0
+GPIO14_A6
+Text Label 5450 6600 2    59   ~ 0
+SCL
+Wire Wire Line
+	5300 5600 5300 5350
+$Comp
+L +3.3V #PWR031
+U 1 1 5A8DCA78
+P 5300 5350
+F 0 "#PWR031" H 5300 5200 50  0001 C CNN
+F 1 "+3.3V" H 5300 5490 50  0000 C CNN
+F 2 "" H 5300 5350 60  0000 C CNN
+F 3 "" H 5300 5350 60  0000 C CNN
+	1    5300 5350
+	1    0    0    -1
+$EndComp
+$Comp
+L GND #PWR032
+U 1 1 5A8DCAEF
+P 5450 5800
+F 0 "#PWR032" H 5450 5550 50  0001 C CNN
+F 1 "GND" H 5450 5650 50  0000 C CNN
+F 2 "" H 5450 5800 60  0000 C CNN
+F 3 "" H 5450 5800 60  0000 C CNN
+	1    5450 5800
+	1    0    0    -1
+$EndComp
+Wire Wire Line
+	5450 5700 5450 5800
+Text Label 5450 6700 2    59   ~ 0
+SDA
+Text Label 5500 3500 0    59   ~ 0
+GPIO16
+Text Label 5500 3400 0    59   ~ 0
+GPIO17
+Text Notes 6000 4850 2    79   ~ 0
+Acceleromter(MPU6050)
+Wire Notes Line
+	4400 4550 4400 7800
 $EndSCHEMATC

Commit message: changed led pad layout
Parts:
- J2: Digikey Part No. (none) -> S7006-ND
Changed lines of the file:
@@
 F 2 "Pin_Headers:Pin_Header_Straight_1x08" H 4900 6000 50  0001 C CNN
 F 3 "" H 4900 6000 50  0001 C CNN
+F 4 "S7006-ND" H 4900 6000 60  0001 C CNN "Digikey Part No."
 	1    4900 6000
 	-1   0    0    1
