File: PCB/pixel/pixel.sch (KiCad schematic (older format))
At the start: 274 parts, among them CON1 BARREL_JACK, P1 CONN_01X04, U1 APA102, U10 APA102, U100 APA102, U101 APA102, U102 APA102, U103 APA102, U104 APA102, U105 APA102, U106 APA102, U107 APA102, U108 APA102, U109 APA102, U11 APA102, U110 APA102, U111 APA102, U112 APA102, U113 APA102, U114 APA102, U115 APA102, U116 APA102, U117 APA102, U118 APA102, U119 APA102, U12 APA102, U120 APA102, U121 APA102, U122 APA102, U123 APA102, U124 APA102, U125 APA102, U126 APA102, U127 APA102, U128 APA102, U129 APA102, U13 APA102, U130 APA102, U131 APA102, U132 APA102, U133 APA102, U134 APA102, U135 APA102, U136 APA102, U137 APA102, U138 APA102, U139 APA102, U14 APA102, U140 APA102, U141 APA102, U142 APA102, U143 APA102, U144 APA102, U145 APA102, U146 APA102, U147 APA102, U148 APA102, U149 APA102, U15 APA102, U150 APA102, U151 APA102, U152 APA102, U153 APA102, U154 APA102, U155 APA102, U156 APA102, U157 APA102, U158 APA102, U159 APA102, U16 APA102, U160 APA102, U161 APA102, U162 APA102, U163 APA102, U164 APA102, U165 APA102, U166 APA102, U167 APA102, U168 APA102, U169 APA102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

Commit message: added fuse, fixed traces
Parts:
- added F1: 5A_Hold, Fuse_Holders_and_Fuses:Fuse_SMD1206_Reflow, symbol Polyfuse_Small
- CON1: Digikey Part No. CP-070BHPJCT-ND -> CP-006APJCT-ND
Connections:
- net +5V: now also F1.1; no longer CON1.1
- new net: CON1.1, F1.2
Changed lines of the file:
@@
 F 2 "idlehands_footprints:DC_POWERJACK_VERT_NoHoles" H 16000 2950 50  0001 C CNN
 F 3 "" H 16000 2950 50  0000 C CNN
-F 4 "CP-070BHPJCT-ND" H 16000 2950 60  0001 C CNN "Digikey Part No."
+F 4 "CP-006APJCT-ND" H 16000 2950 60  0001 C CNN "Digikey Part No."
 	1    16000 2950
 	1    0    0    -1
 $EndComp
 Wire Wire Line
-	16300 2850 16350 2850
-Wire Wire Line
-	16350 2850 16350 2700
+	16300 2850 16550 2850
 Wire Wire Line
 	16300 3050 16350 3050
@@
 L +5V #PWR036
 U 1 1 5A67DCE4
-P 16350 2700
-F 0 "#PWR036" H 16350 2550 50  0001 C CNN
-F 1 "+5V" H 16350 2840 50  0000 C CNN
-F 2 "" H 16350 2700 50  0000 C CNN
-F 3 "" H 16350 2700 50  0000 C CNN
-	1    16350 2700
+P 16900 2650
+F 0 "#PWR036" H 16900 2500 50  0001 C CNN
+F 1 "+5V" H 16900 2790 50  0000 C CNN
+F 2 "" H 16900 2650 50  0000 C CNN
+F 3 "" H 16900 2650 50  0000 C CNN
+	1    16900 2650
 	1    0    0    -1
 $EndComp
@@
 Wire Wire Line
 	18900 6100 18900 6050
+$Comp
+L Polyfuse_Small F1
+U 1 1 5A8EE8CE
+P 16650 2850
+F 0 "F1" V 16575 2850 50  0000 C CNN
+F 1 "5A_Hold" V 16725 2850 50  0000 C CNN
+F 2 "Fuse_Holders_and_Fuses:Fuse_SMD1206_Reflow" H 16700 2650 50  0001 L CNN
+F 3 "" H 16650 2850 50  0001 C CNN
+F 4 "MF-USML400-2CT-ND" V 16650 2850 60  0001 C CNN "Digikey Part No."
+	1    16650 2850
+	0    1    1    0
+$EndComp
+Wire Wire Line
+	16750 2850 16900 2850
+Wire Wire Line
+	16900 2850 16900 2650
 $EndSCHEMATC

Commit message: changed led pad layout
Parts:
- U1, U10, U100, U101, U102, U103, U104, U105, U106, U107, U108, U109, U11, U110, U111, U112, U113, U114, U115, U116, U117, U118, U119, U12, U120, U121, U122, U123, U124, U125, U126, U127, U128, U129, U13, U130, U131, U132, U133, U134, U135, U136, U137, U138, U139, U14, U140, U141, U142, U143, U144, U145, U146, U147, U148, U149, U15, U150, U151, U152, U153, U154, U155, U156, U157, U158, U159, U16, U160, U161, U162, U163, U164, U165, U166, U167, U168, U169, U17, U170, U171, U172, U173, U174, U175, U176, U177, U178, U179, U18, U180, U181, U182, U183, U184, U185, U186, U187, U188, U189, U19, U190, U191, U192, U193, U194, U195, U196, U197, U198, U199, U2, U20, U200, U201, U202, U203, U204, U205, U206, U207, U208, U209, U21, U210, U211, U212, U213, U214, U215, U216, U217, U218, U219, U22, U220, U221, U222, U223, U224, U225, U226, U227, U228, U229, U23, U230, U231, U232, U233, U234, U235, U236, U237, U238, U239, U24, U240, U241, U242, U243, U244, U245, U246, U247, U248, U249, U25, U250, U251, U252, U253, U254, U255, U256, U26, U27, U28, U29, U3, U30, U31, U32, U33, U34, U35, U36, U37, U38, U39, U4, U40, U41, U42, U43, U44, U45, U46, U47, U48, U49, U5, U50, U51, U52, U53, U54, U55, U56, U57, U58, U59, U6, U60, U61, U62, U63, U64, U65, U66, U67, U68, U69, U7, U70, U71, U72, U73, U74, U75, U76, U77, U78, U79, U8, U80, U81, U82, U83, U84, U85, U86, U87, U88, U89, U9, U90, U91, U92, U93, U94, U95, U96, U97, U98, U99: footprint idlehands_footprints:APA102-2020_NOGND -> idlehands_footprints:APA102-2020_AFSTYLE

Commit message: LED Layout Modified
Parts:
- F1: Digikey Part No. MF-USML400-2CT-ND -> MF-USML500-2CT-ND
Changed lines of the file:
@@
 F 2 "Fuse_Holders_and_Fuses:Fuse_SMD1206_Reflow" H 16700 2650 50  0001 L CNN
 F 3 "" H 16650 2850 50  0001 C CNN
-F 4 "MF-USML400-2CT-ND" V 16650 2850 60  0001 C CNN "Digikey Part No."
+F 4 "MF-USML500-2CT-ND" V 16650 2850 60  0001 C CNN "Digikey Part No."
 	1    16650 2850
 	0    1    1    0
